File: schematic/D-SP-X1-01-A.sch (EAGLE design)
At the start: 1 part

Commit message: Updated schematic.
Parts:
- added C1: -, rcl:C-EUC0603
- added C4: 1uF, rcl:C-EUC0603
- added C5, C6, C7: 100n, rcl:C-EUC0603
- added C8: 10n, rcl:C-EUC0603
- added CD1: 4.7uF/400v, rcl:CPOL-EUE2.5-6
- added CD2: 1uF/400v, rcl:CPOL-EUE2.5-6
- added CD3: 330uF / 6.3v, rcl:CPOL-EUE2.5-6
- added D1, D3, D4, D9: (no value), diode:DIODE-SCD80-INFINEON
- added D10, D7: (no value), led:LEDCHIP-LED0603
- added D8: 0R, rcl:R-EU_R0603
- added FR1: "Fuse" MELF, fuse:FUSELITTLEFUSE
- added FR2: 10A/250V, fuse:FUSELITTLEFUSE
- added IN, OUT: (no value), con-phoenix-254:MPT2
- added K1: AZ8-FORM-A, relay:AZ8-FORM-A
- added L1, L2: 1mH, rcl:L-EU0204V
- added Q1, Q2: (no value), transistor:BC850-NPN-SOT23-BEC
- added R1: 8k2, rcl:R-EU_R0603
- added R10, R14, R19, R5: 2k2, rcl:R-EU_R0603
- added R11, R13, R6, R7: 10k, rcl:R-EU_R0603
- added R12, R8: 470k, rcl:R-EU_R1206
- added R2: 3k3, rcl:R-EU_R0603
- added R3: MOV, rcl:R-EU_R1206
- added R4: 43k, rcl:R-EU_R0603
- added R9: NTC100K, rcl:R-EU_R0603
- added RX, TX, VDD_3.3V: TPTP17R, testpad:TPTP17R
- added SW1, SW2: (no value), switch-omron:10-XX
Connections:
- new net +3V3: C4.1, CD3.+, R4.1, R6.2, R7.2, U$1.VDD, VDD_3.3V.TP
- new net +5V: D8.1, K1K.1, R1.2
- new net GND: C4.2, C5.2, C6.2, C7.2, C8.2, CD1.-, CD2.-, CD3.-, D10.C, D3.A, D7.C, D9.A, Q1.E, Q2.E, R11.2, R13.2, R3.1, R9.2, SW1.P, SW1.P1, SW2.S, SW2.S1, U$1.GND@0, U$1.GND@1
- new net L: FR1.1, FR2.1, IN-2.1
- new net LED_ERROR: R5.2, U$1.PD01
- new net LED_STATUS: R19.2, U$1.PC04
- new net N: IN-1.1
- new net N$1: RX.TP, U$1.PC00
- new net N$10: Q2.C, R13.1, R14.2
- new net N$11: FR2.2, K1-1.P, R8.1
- new net N$12: K1-1.S, OUT-1.1
- new net N$13: D1.A, FR1.2, R3.2
- new net N$14: CD1.+, D1.C, L1.1
- new net N$15: CD2.+, L1.2
- new net N$16: C1.2, L2.2, R2.2
- new net N$17: C1.1
- new net N$18: R1.1, R2.1
- new net N$19: D3.C, L2.1
- new net N$2: TX.TP, U$1.PC01
- new net N$3: D10.A, R19.1
- new net N$4: D7.A, R5.1
- new net N$5: Q1.B, R10.1, R11.1
- new net N$6: D4.A, K1K.2, Q1.C
- new net N$7: D4.C, D8.2
- new net N$8: R12.1, R8.2
- new net N$9: D9.C, Q2.B, R12.2
- new net PAIR/50HZ_DETECT: C6.1, C8.1, R14.1, R6.1, SW1.S, SW1.S1, U$1.PA03, U$1.PA04
- new net RELAY: R10.2, U$1.PC03
- new net RELAY_TEMP: C5.1, R4.2, R9.1, U$1.PC02
- new net SWITCH: C7.1, R7.1, SW2.P, SW2.P1, U$1.PC05
Other:
- note added: "3.3V Regulator"
- note added: "504.638.80"
- note added: "50HZ feedback/fuse check"
- note added: "Mikael Sundin"
- note added: "N"
- note added: "R9 Close to Relay"
- note added: "STEP DOWN PB8516 (Similar to BP8519C)"
- note added: "www.linkedin.com/in/mikaelsundin"
- note added: "Åskväder Zigbee Relay"

Commit message: Updated schematic with zigbee module model name.
Other:
- note added: "MGM210L"
Changed lines of the file:
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@@
 <setting verticaltext="up"/>
 </settings>
-<grid distance="100" unitdist="mil" unit="mil" style="lines" multiple="1" display="no" altdistance="0.01" altunitdist="inch" altunit="inch"/>
+<grid distance="50" unitdist="mil" unit="mil" style="lines" multiple="1" display="no" altdistance="0.01" altunitdist="inch" altunit="inch"/>
 <layers>
-<layer number="1" name="Top" color="4" fill="1" visible="yes" active="no"/>
-<layer number="16" name="Bottom" color="1" fill="1" visible="yes" active="no"/>
-<layer number="17" name="Pads" color="2" fill="1" visible="yes" active="no"/>
-<layer number="18" name="Vias" color="2" fill="1" visible="yes" active="no"/>
-<layer number="19" name="Unrouted" color="6" fill="1" visible="yes" active="no"/>
-<layer number="20" name="Dimension" color="24" fill="1" visible="yes" active="no"/>
-<layer number="21" name="tPlace" color="7" fill="1" visible="yes" active="no"/>
-<layer number="22" name="bPlace" color="7" fill="1" visible="yes" active="no"/>
-<layer number="23" name="tOrigins" color="15" fill="1" visible="yes" active="no"/>
-<layer number="24" name="bOrigins" color="15" fill="1" visible="yes" active="no"/>
-<layer number="25" name="tNames" color="7" fill="1" visible="yes" active="no"/>
-<layer number="26" name="bNames" color="7" fill="1" visible="yes" active="no"/>
-<layer number="27" name="tValues" color="7" fill="1" visible="yes" active="no"/>
-<layer number="28" name="bValues" color="7" fill="1" visible="yes" active="no"/>
+<layer number="1" name="Top" color="4" fill="1" visible="no" active="no"/>
+<layer number="16" name="Bottom" color="1" fill="1" visible="no" active="no"/>
+<layer number="17" name="Pads" color="2" fill="1" visible="no" active="no"/>
+<layer number="18" name="Vias" color="2" fill="1" visible="no" active="no"/>
+<layer number="19" name="Unrouted" color="6" fill="1" visible="no" active="no"/>
+<layer number="20" name="Dimension" color="24" fill="1" visible="no" active="no"/>
+<layer number="21" name="tPlace" color="7" fill="1" visible="no" active="no"/>
+<layer number="22" name="bPlace" color="7" fill="1" visible="no" active="no"/>
+<layer number="23" name="tOrigins" color="15" fill="1" visible="no" active="no"/>
+<layer number="24" name="bOrigins" color="15" fill="1" visible="no" active="no"/>
+<layer number="25" name="tNames" color="7" fill="1" visible="no" active="no"/>
+<layer number="26" name="bNames" color="7" fill="1" visible="no" active="no"/>
+<layer number="27" name="tValues" color="7" fill="1" visible="no" active="no"/>
+<layer number="28" name="bValues" color="7" fill="1" visible="no" active="no"/>
 <layer number="29" name="tStop" color="7" fill="3" visible="no" active="no"/>
 <layer number="30" name="bStop" color="7" fill="6" visible="no" active="no"/>
@@
 <layer number="35" name="tGlue" color="7" fill="4" visible="no" active="no"/>
 <layer number="36" name="bGlue" color="7" fill="5" visible="no" active="no"/>
-<layer number="37" name="tTest" color="7" fill="1" visible="yes" active="no"/>
-<layer number="38" name="bTest" color="7" fill="1" visible="yes" active="no"/>
+<layer number="37" name="tTest" color="7" fill="1" visible="no" active="no"/>
+<layer number="38" name="bTest" color="7" fill="1" visible="no" active="no"/>
 <layer number="39" name="tKeepout" color="4" fill="11" visible="no" active="no"/>
 <layer number="40" name="bKeepout" color="1" fill="11" visible="no" active="no"/>
@@
 <layer number="44" name="Drills" color="7" fill="1" visible="no" active="no"/>
 <layer number="45" name="Holes" color="7" fill="1" visible="no" active="no"/>
-<layer number="46" name="Milling" color="3" fill="1" visible="yes" active="no"/>
-<layer number="47" name="Measures" color="7" fill="1" visible="yes" active="no"/>
-<layer number="48" name="Document" color="7" fill="1" visible="yes" active="no"/>
-<layer number="49" name="Reference" color="7" fill="1" visible="yes" active="no"/>
-<layer number="51" name="tDocu" color="7" fill="1" visible="yes" active="no"/>
-<layer number="52" name="bDocu" color="7" fill="1" visible="yes" active="no"/>
+<layer number="46" name="Milling" color="3" fill="1" visible="no" active="no"/>
+<layer number="47" name="Measures" color="7" fill="1" visible="no" active="no"/>
+<layer number="48" name="Document" color="7" fill="1" visible="no" active="no"/>
+<layer number="49" name="Reference" color="7" fill="1" visible="no" active="no"/>
+<layer number="51" name="tDocu" color="7" fill="1" visible="no" active="no"/>
+<layer number="52" name="bDocu" color="7" fill="1" visible="no" active="no"/>
 <layer number="88" name="SimResults" color="9" fill="1" visible="yes" active="yes"/>
 <layer number="89" name="SimProbes" color="9" fill="1" visible="yes" active="yes"/>
@@
 <text x="216.916" y="20.32" size="3.048" layer="91">504.638.80</text>
 <text x="162.306" y="19.558" size="3.048" layer="91">Åskväder Zigbee Relay</text>
+<text x="133.35" y="140.97" size="3.81" layer="97" align="center">MGM210L</text>
 </plain>
 <instances>
